File: kicad/swd-adapter/swd-adapter.kicad_pcb (KiCad board)
At the start: 2 copper layers, 10 x 22.3 mm, 4 parts, among them SW1 swd_connector_2_45, SW2 swd_connector_1_27

Commit message: added pour
Routing:
- added copper zone on B.Cu, net (none)
- added copper zone on F.Cu, net (none)
Changed lines of the file:
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@@
       (effects (font (size 1 1) (thickness 0.15)))
     )
+    (fp_circle (center 0 0) (end 2.45 0) (layer F.CrtYd) (width 0.05))
+    (fp_circle (center 0 0) (end 2.2 0) (layer Cmts.User) (width 0.15))
     (fp_text user %R (at 0.3 0) (layer F.Fab)
       (effects (font (size 1 1) (thickness 0.15)))
     )
-    (fp_circle (center 0 0) (end 2.2 0) (layer Cmts.User) (width 0.15))
-    (fp_circle (center 0 0) (end 2.45 0) (layer F.CrtYd) (width 0.05))
     (pad 1 thru_hole circle (at 1.166726 -1.166726) (size 0.7 0.7) (drill 0.4) (layers *.Cu *.Mask))
     (pad 1 thru_hole circle (at 0 -1.65) (size 0.7 0.7) (drill 0.4) (layers *.Cu *.Mask))
@@
   (segment (start 158.73 105.83) (end 157.2 104.3) (width 0.25) (layer B.Cu) (net 2))
   (segment (start 158.73 110) (end 158.73 105.83) (width 0.25) (layer B.Cu) (net 2))
-  (segment (start 156.4 93.06) (end 157.46 92) (width 0.25) (layer F.Cu) (net 3))
-  (segment (start 156.4 103.9) (end 156.4 93.06) (width 0.25) (layer F.Cu) (net 3))
-  (segment (start 158.73 106.23) (end 156.4 103.9) (width 0.25) (layer F.Cu) (net 3))
+  (segment (start 156.5 92.96) (end 157.46 92) (width 0.25) (layer F.Cu) (net 3))
+  (segment (start 156.5 104) (end 156.5 92.96) (width 0.25) (layer F.Cu) (net 3))
+  (segment (start 158.73 106.23) (end 156.5 104) (width 0.25) (layer F.Cu) (net 3))
   (segment (start 158.73 110) (end 158.73 106.23) (width 0.25) (layer F.Cu) (net 3))
   (segment (start 160 98.6) (end 160 92) (width 0.25) (layer F.Cu) (net 4))
@@
   (segment (start 161.27 106.43) (end 163.365001 104.334999) (width 0.25) (layer F.Cu) (net 5))
   (segment (start 161.27 110) (end 161.27 106.43) (width 0.25) (layer F.Cu) (net 5))
+  (zone (net 0) (net_name "") (layer F.Cu) (hatch edge 0.508)
+    (connect_pads (clearance 0.508))
+    (min_thickness 0.254)
+    (fill yes (arc_segments 32) (thermal_gap 0.508) (thermal_bridge_width 0.508))
+    (polygon
+      (pts
+        (xy 165.5 112) (xy 154.5 112) (xy 154.5 88.5) (xy 165.5 88.5)
+      )
+    )
+  )
+  (zone (net 0) (net_name "") (layer B.Cu) (hatch edge 0.508)
+    (connect_pads (clearance 0.508))
+    (min_thickness 0.254)
+    (fill yes (arc_segments 32) (thermal_gap 0.508) (thermal_bridge_width 0.508))
+    (polygon
+      (pts
+        (xy 165.5 112) (xy 154.5 112) (xy 154.5 88.5) (xy 165.5 88.5)
+      )
+    )
+  )
 )
